File: Temps_South_DCT_HSK/Temps_South_DCT_HSK.kicad_pcb (KiCad board)
At the start: 2 copper layers, 53.3 x 57.1 mm, 7 parts, among them J1 North_Temps_1, J2 North_Temps_2, J3 Internal_Temps_DCT_HSK_Box_1, J4 Internal_Temps_DCT_HSK_Box_2

Commit message: See previous commit
Parts:
- added REF**: MountingHole_3.2mm_M3, MountingHole:MountingHole_3.2mm_M3, F.Cu at (114.2, 75.6)
- added REFe: MountingHole_3.2mm_M3, MountingHole:MountingHole_3.2mm_M3, F.Cu at (122.8, 75.6)
- moved G*** 0.13 mm to (129.0, 75.5)
Other:
- board text added: "Temps South Rev B Dennis H. Calderon 09/09/2023"
- board text removed: "Temps_South_DCT_HSK Dennis H. Calderon 01/23/2023"
