File: Temps_South/Temps_South.kicad_pcb (KiCad board)
At the start: 2 copper layers, 53.3 x 57.1 mm, 9 parts, among them J1 North_Temps_1, J2 North_Temps_2, J3 Internal_Temps_DCT_HSK_Box_1, J4 Internal_Temps_DCT_HSK_Box_2

Commit message: Added mounting holes for North Temp. South Temp board updated based off K. McBride pull request.
Parts:
- removed the G*** at (130.0, 53.5)
- added G***: Stormtrooper, Fun_Logos:Stormtrooper, F.Cu at (130.0, 53.5)
Other:
- board text added: "STB1"
- board text added: "STB2"
- board text added: "South"
- board text added: "Temps South Rev B Dennis H. Calderon 09/09/2023"
- board text removed: "NTB1"
- board text removed: "NTB2"
- board text removed: "North"
- board text removed: "Temps North Rev B Dennis H. Calderon 09/09/2023"

Commit message: Updated Heater South with correct mapping referencing DCT_Heater_Driver schematic. Updated silscreen on all boards. Generated fabrication files.
Changed lines of the file:
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@@
       (drillshape 0)
       (scaleselection 1)
-      (outputdirectory "Fab")
+      (outputdirectory "Fab/Rev_B")
     )
   )
@@
     (at 130.010943 53.524623)
     (attr board_only exclude_from_pos_files exclude_from_bom)
-    (fp_text reference "G***" (at 0 0) (layer "F.SilkS")
+    (fp_text reference "G***" (at 0 0) (layer "F.SilkS") hide
         (effects (font (size 1.524 1.524) (thickness 0.3)))
     )
@@
       (stroke (width 0) (type solid)) (fill solid) (layer "B.SilkS"))
   )
+  (gr_circle (center 138.8364 79.8322) (end 138.8618 79.8322)
+    (stroke (width 0.254) (type solid)) (fill none) (layer "B.SilkS"))
   (gr_circle (center 92.680001 50.83) (end 92.680002 50.83)
     (stroke (width 0.254) (type solid)) (fill none) (layer "B.SilkS"))
   (gr_circle (center 92.69 80.02) (end 92.690001 80.02)
     (stroke (width 0.254) (type solid)) (fill none) (layer "B.SilkS"))
-  (gr_circle (center 138.29 50.9) (end 138.392956 50.9)
+  (gr_circle (center 138.8364 50.9) (end 138.8618 50.9)
+    (stroke (width 0.254) (type solid)) (fill none) (layer "B.SilkS"))
+  (gr_circle (center 138.8364 50.9) (end 138.8618 50.9)
     (stroke (width 0.254) (type solid)) (fill none) (layer "F.SilkS"))
   (gr_circle (center 92.67 50.83) (end 92.670001 50.83)
@@
   (gr_circle (center 92.68 80.02) (end 92.680001 80.02)
     (stroke (width 0.254) (type solid)) (fill none) (layer "F.SilkS"))
-  (gr_circle (center 138.21 79.92) (end 138.312956 79.92)
+  (gr_circle (center 138.8364 79.8322) (end 138.8618 79.8322)
     (stroke (width 0.254) (type solid)) (fill none) (layer "F.SilkS"))
   (gr_line (start 118.11 43.4848) (end 118.11 106.5276)

Commit message: I was working towards fabrication. Chaged the KiCAD violation issues for each PCB to run all tests and make some important silkscreen font bigger. I also edited a few traces and even removed a few vias to make the trace clearance to the edge of the PCBs larger. Need to add the correct centers for the 34-pin connectors on each PCB, rerun traces, and then we should be good.
Changed lines of the file:
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@@
     (grid_origin 122.7074 53.1876)
     (pcbplotparams
-      (layerselection 0x00010fc_ffffffff)
+      (layerselection 0x003d0ff_ffffffff)
       (plot_on_all_layers_selection 0x0000000_00000000)
       (disableapertmacros false)
@@
       (drillshape 0)
       (scaleselection 1)
-      (outputdirectory "Fab/Rev_B")
+      (outputdirectory "Fab/Rev_B/")
     )
   )
@@
   (gr_rect (start 91.44 46.99) (end 144.78 104.14)
     (stroke (width 0.1) (type solid)) (fill none) (layer "Edge.Cuts"))
+  (gr_text "Temps South Rev B\nDennis H. Calderon\n09/09/2023" (at 127.2074 99.3876) (layer "B.SilkS")
+    (effects (font (size 1.3 1.3) (thickness 0.3) bold) (justify mirror))
+  )
   (gr_text "South" (at 129.123619 50.5376) (layer "B.SilkS")
     (effects (font (size 3.5 3.5) (thickness 0.5)) (justify mirror))
@@
     (effects (font (size 2.5 2.5) (thickness 0.4)))
   )
-  (gr_text "Temps South Rev B\nDennis H. Calderon\n09/09/2023" (at 127.3074 101.7626) (layer "F.SilkS")
-    (effects (font (size 0.762 0.762) (thickness 0.15)))
-  )
   (gr_text "STB2\n" (at 100.1824 90.017601 90) (layer "F.SilkS")
-    (effects (font (size 1 1) (thickness 0.2)))
+    (effects (font (size 1.5 1.5) (thickness 0.3) bold))
   )
   (gr_text "STB2" (at 136.3074 89.9876 90) (layer "F.SilkS")
-    (effects (font (size 1 1) (thickness 0.2)))
+    (effects (font (size 1.3 1.3) (thickness 0.3) bold))
   )
   (gr_text "From DCT" (at 102.8574 75.7626 -270) (layer "F.SilkS")
@@
   )
   (gr_text "STB1" (at 136.3074 61.112401 90) (layer "F.SilkS")
-    (effects (font (size 1 1) (thickness 0.2)))
+    (effects (font (size 1.5 1.5) (thickness 0.3) bold))
   )
   (gr_text "STB1" (at 100.1824 61.061601 90) (layer "F.SilkS")
-    (effects (font (size 1 1) (thickness 0.2)))
+    (effects (font (size 1.5 1.5) (thickness 0.3) bold))
+  )
+  (dimension (type aligned) (layer "Edge.Cuts")
+    (pts (xy 144.78 104.14) (xy 144.78 46.99))
+    (height 3.5274)
+    (gr_text "57.1500 mm" (at 147.1574 75.565 90) (layer "Edge.Cuts")
+      (effects (font (size 1 1) (thickness 0.15)))
+    )
+    (format (prefix "") (suffix "") (units 3) (units_format 1) (precision 4))
+    (style (thickness 0.1) (arrow_length 1.27) (text_position_mode 0) (extension_height 0.58642) (extension_offset 0.5) keep_text_aligned)
+  )
+  (dimension (type aligned) (layer "Edge.Cuts")
+    (pts (xy 144.78 46.99) (xy 91.44 46.99))
+    (height 2.002399)
+    (gr_text "53.3400 mm" (at 118.11 43.837601) (layer "Edge.Cuts")
+      (effects (font (size 1 1) (thickness 0.15)))
+    )
+    (format (prefix "") (suffix "") (units 3) (units_format 1) (precision 4))
+    (style (thickness 0.1) (arrow_length 1.27) (text_position_mode 0) (extension_height 0.58642) (extension_offset 0.5) keep_text_aligned)
   )
   (segment (start 139.0074 48.8876) (end 140.8074 50.6876) (width 0.2) (layer "F.Cu") (net 3))
@@
   (segment (start 127.4414 71.2216) (end 96.52 71.2216) (width 0.2) (layer "B.Cu") (net 32))
   (segment (start 130.4074 74.1876) (end 127.4414 71.2216) (width 0.2) (layer "B.Cu") (net 32))
-  (segment (start 122.6074 78.7876) (end 123.6774 79.8576) (width 0.2) (layer "F.Cu") (net 33))
-  (segment (start 93.94444 79.8576) (end 93.94444 79.65056) (width 0.2) (layer "F.Cu") (net 33))
-  (segment (start 94.8074 78.7876) (end 122.6074 78.7876) (width 0.2) (layer "F.Cu") (net 33))
-  (segment (start 123.6774 79.8576) (end 139.65984 79.8576) (width 0.2) (layer "F.Cu") (net 33))
   (segment (start 93.94444 79.65056) (end 94.8074 78.7876) (width 0.2) (layer "F.Cu") (net 33))
+  (segment (start 138.58984 78.7876) (end 139.65984 79.8576) (width 0.2) (layer "F.Cu") (net 33))
+  (segment (start 94.8074 78.7876) (end 138.58984 78.7876) (width 0.2) (layer "F.Cu") (net 33))
+  (segment (start 93.94444 79.8576) (end 93.94444 79.65056) (width 0.2) (layer "F.Cu") (net 33))
   (segment (start 139.530403 79.987037) (end 139.65984 79.8576) (width 0.2) (layer "F.Cu") (net 33))
-  (segment (start 110.8074 77.4876) (end 139.85016 77.4876) (width 0.2) (layer "B.Cu") (net 34))
-  (segment (start 108.4374 79.8576) (end 110.8074 77.4876) (width 0.2) (layer "B.Cu") (net 34))
+  (segment (start 96.5374 79.8576) (end 98.9074 77.4876) (width 0.2) (layer "B.Cu") (net 34))
   (segment (start 139.85016 77.4876) (end 142.22016 79.8576) (width 0.2) (layer "B.Cu") (net 34))
-  (segment (start 96.50476 79.8576) (end 108.4374 79.8576) (width 0.2) (layer "B.Cu") (net 34))
+  (segment (start 98.9074 77.4876) (end 139.85016 77.4876) (width 0.2) (layer "B.Cu") (net 34))
+  (segment (start 96.50476 79.8576) (end 96.5374 79.8576) (width 0.2) (layer "B.Cu") (net 34))
   (segment (start 96.50476 79.8576) (end 96.67476 79.6876) (width 0.2) (layer "B.Cu") (net 34))
-  (segment (start 93.8074 77.9876) (end 124.0074 77.9876) (width 0.2) (layer "F.Cu") (net 37))
-  (segment (start 124.0074 77.9876) (end 124.4074 78.3876) (width 0.2) (layer "F.Cu") (net 37))
-  (segment (start 140.7074 81.3602) (end 139.67 82.3976) (width 0.2) (layer "F.Cu") (net 37))
   (segment (start 140.7074 79.0876) (end 140.7074 81.3602) (width 0.2) (layer "F.Cu") (net 37))
+  (segment (start 93.9546 82.3976) (end 93.0074 81.4504) (width 0.2) (layer "F.Cu") (net 37))
+  (segment (start 93.8074 77.9876) (end 139.6074 77.9876) (width 0.2) (layer "F.Cu") (net 37))
+  (segment (start 139.6074 77.9876) (end 140.7074 79.0876) (width 0.2) (layer "F.Cu") (net 37))
+  (segment (start 140.7074 81.3602) (end 139.67 82.3976) (width 0.2) (layer "F.Cu") (net 37))
   (segment (start 93.0074 78.7876) (end 93.8074 77.9876) (width 0.2) (layer "F.Cu") (net 37))
   (segment (start 93.0074 81.4504) (end 93.0074 78.7876) (width 0.2) (layer "F.Cu") (net 37))
-  (segment (start 124.4074 78.3876) (end 140.0074 78.3876) (width 0.2) (layer "F.Cu") (net 37))
-  (segment (start 140.0074 78.3876) (end 140.7074 79.0876) (width 0.2) (layer "F.Cu") (net 37))
-  (segment (start 93.9546 82.3976) (end 93.0074 81.4504) (width 0.2) (layer "F.Cu") (net 37))
-  (segment (start 140.8074 80.995) (end 140.8074 79.1876) (width 0.2) (layer "B.Cu") (net 38))
+  (segment (start 140.1074 78.4876) (end 100.3074 78.4876) (width 0.2) (layer "B.Cu") (net 38))
   (segment (start 142.21 82.3976) (end 140.8074 80.995) (width 0.2) (layer "B.Cu") (net 38))
+  (segment (start 140.8074 80.995) (end 140.8074 79.1876) (width 0.2) (layer "B.Cu") (net 38))
+  (segment (start 100.3074 78.4876) (end 96.4946 82.3004) (width 0.2) (layer "B.Cu") (net 38))
   (segment (start 140.8074 79.1876) (end 140.1074 78.4876) (width 0.2) (layer "B.Cu") (net 38))
-  (segment (start 112.2074 78.4876) (end 108.2974 82.3976) (width 0.2) (layer "B.Cu") (net 38))
-  (segment (start 108.2974 82.3976) (end 96.4946 82.3976) (width 0.2) (layer "B.Cu") (net 38))
   (segment (start 142.21 82.3976) (end 141.9174 82.3976) (width 0.2) (layer "B.Cu") (net 38))
-  (segment (start 140.1074 78.4876) (end 112.2074 78.4876) (width 0.2) (layer "B.Cu") (net 38))
+  (segment (start 96.4946 82.3004) (end 96.4946 82.3976) (width 0.2) (layer "B.Cu") (net 38))
   (segment (start 141.1074 78.921915) (end 141.1074 83.835) (width 0.2) (layer "F.Cu") (net 41))
   (segment (start 111.2074 76.4876) (end 111.969909 76.4876) (width 0.2) (layer "F.Cu") (net 41))
